File: dectspansion.kicad_pcb (KiCad board)
At the start: 4 copper layers, 37 x 36.6 mm, 18 parts, among them J1 Hexpansion-Connector, J3 AudioJack4, U2 SC14CVMDECT

Commit message: Created PCB layout
Parts:
- added J2: Conn_01x03_Pin, Connector_PinHeader_2.54mm:PinHeader_1x03_P2.54mm_Vertical, F.Cu at (108.5, 92.0)
- moved JP1 13.7 mm to (107.6, 107.7), turned to -90 degrees
- moved R6 5.29 mm to (118.0, 96.7), turned to -90 degrees
- moved C4 1.47 mm to (116.2, 96.9)
- moved C9 1.47 mm to (112.4, 96.7)
- moved C6 1.47 mm to (114.2, 96.9)
- moved C5 1.47 mm to (110.6, 96.9)
- moved J3 0.29 mm to (126.1, 87.8)
Routing:
- net GND: track 61.5 -> 76.5 mm, vias 12 -> 14
- net /HS_I: track 23.3 -> 34.6 mm
- net /HS_H: track 24.0 -> 35.2 mm
- net /HEXP_DET: track 17.2 -> 11.3 mm
- net Net-(U2-CHARGE): track 2.66 -> 8.45 mm, vias 0 -> 2
- net +3V3: track 56.7 -> 51.5 mm
